Commit message: reconfigured joints

File: vscode/my-robot/robot.urdf (robot description, URDF)
Before this commit: robot onshape, 3 links, 2 joints
Links:
- removed link wheel
- removed link wheel_2
- added link assembly_3, mass 0.043528139347743959042; collision mesh filename=package:///jgy-370output_shaft.stl; collision mesh filename=package:///part_1.stl
- added link assembly_3_2, mass 0.043528139347743959042; collision mesh filename=package:///jgy-370output_shaft.stl; collision mesh filename=package:///part_1.stl
- added link idler, mass 0.020048491397287253324; collision mesh filename=package:///shaft2.stl; collision mesh filename=package:///spur_gear13.stl
- added link idler_2, mass 0.020048491397287253324; collision mesh filename=package:///shaft2.stl; collision mesh filename=package:///spur_gear13.stl
- added link idler_3, mass 0.020048491397287253324; collision mesh filename=package:///shaft2.stl; collision mesh filename=package:///spur_gear13.stl
- added link idler_4, mass 0.020048491397287253324; collision mesh filename=package:///shaft2.stl; collision mesh filename=package:///spur_gear13.stl
- added link lim_frame, mass 0.13451687861695468817; collision mesh filename=package:///frame.stl; collision mesh filename=package:///frame.stl
- added link lim_frame_2, mass 0.13451687861695471593; collision mesh filename=package:///frame.stl; collision mesh filename=package:///frame.stl
- added link wheel_shaft, mass 0.077205002433972699794; collision mesh filename=package:///m5-nut-4mm.stl; collision mesh filename=package:///m5-nut-4mm.stl
- added link wheel_shaft_2, mass 0.077205002433972699794; collision mesh filename=package:///m5-nut-4mm.stl; collision mesh filename=package:///m5-nut-4mm.stl
- added link wheel_shaft_3, mass 0.077205002433972699794; collision mesh filename=package:///m5-nut-4mm.stl; collision mesh filename=package:///m5-nut-4mm.stl
- added link wheel_shaft_4, mass 0.077205002433972699794; collision mesh filename=package:///m5-nut-4mm.stl; collision mesh filename=package:///m5-nut-4mm.stl
- link body: mass 2.2387448144601149735 -> 0.93999623980613211671; geometry collision mesh filename=package:///back_plate.stl; collision mesh filename=package:///bottom_plate.stl
Joints:
- removed joint wheel1_speed
- removed joint wheel2_speed
- added joint idler_a: type revolute, parent lim_frame_2, child idler_3, origin xyz=0.069999999999997036815 0 0.00800000000000022915 rpy=2.05761454752299006e-15 -1.7554786218493166925e-15 2.3580333328824618633, axis 0 0 1, limit effort=1 velocity=20
- added joint idler_b: type revolute, parent lim_frame_2, child idler_4, origin xyz=-0.06999999999999706457 2.7755575615628913511e-16 0.0080000000000000903722 rpy=2.8375496426252807701e-16 2.075297764247214519e-15 -2.5897213190487309298, axis 0 0 1, limit effort=1 velocity=20
- added joint idler_c: type revolute, parent lim_frame, child idler, origin xyz=0.070000000000000228706 2.2204460492503130808e-16 0.0079999999999996879163 rpy=-1.4164323340577334528e-15 3.7025772151567372099e-15 2.6685569241801592177, axis 0 0 1, limit effort=1 velocity=20
- added joint idler_d: type revolute, parent lim_frame, child idler_2, origin xyz=-0.06999999999999995115 1.1657341758564143674e-15 0.0079999999999999793499 rpy=7.1568118488118355445e-16 1.0327968037644009249e-16 2.2680270748056519103, axis 0 0 1, limit effort=1 velocity=20
- added joint motor_a: type revolute, parent body, child assembly_3_2, origin xyz=-0.31888221975469926983 0.18552361240918216478 0.25494999775085969151 rpy=-1.5607748743761082899 -9.08699813967281389e-05 -3.1234578701676607437, axis 0 0 1, limit effort=1 velocity=20
- added joint motor_b: type revolute, parent body, child assembly_3, origin xyz=-0.31783952686720584602 0.12803595497214695365 0.25552622161746796348 rpy=3.1325252042406694919 1.5607744624144965773 -1.5617285373929443715, axis 0 0 1, limit effort=1 velocity=20
- added joint sun_a: type revolute, parent assembly_3_2, child lim_frame_2, origin xyz=-2.2204460492503130808e-16 0.00010468429334425932709 -0.028999999999999914735 rpy=3.1415926535897926719 -2.8669353829452643957e-16 -3.1415926535897886751, axis 0 0 1, limit effort=1 velocity=20
- added joint sun_b: type revolute, parent assembly_3, child lim_frame, origin xyz=1.6653345369377348106e-16 0.00010468429334442586054 -0.02899999999999994249 rpy=-3.1415926535897917837 3.3251181200224165922e-16 1.3010147677694188229, axis 0 0 1, limit effort=1 velocity=20
- added joint wheel_a: type revolute, parent lim_frame_2, child wheel_shaft_3, origin xyz=0.1109999999999954079 5.5511151231257827021e-17 0.0080000000000000071054 rpy=1.2500110860542346747e-15 -1.544204936456279263e-15 -2.7410493356107226148, axis 0 0 1, limit effort=1 velocity=20
- added joint wheel_b: type revolute, parent lim_frame_2, child wheel_shaft_4, origin xyz=-0.11099999999999532463 2.7755575615628913511e-16 0.0079999999999999793499 rpy=1.2736879123411381812e-15 2.5288747077123325142e-15 1.8176008417319950983, axis 0 0 1, limit effort=1 velocity=20
- added joint wheel_c: type revolute, parent lim_frame, child wheel_shaft, origin xyz=0.11100000000000004308 0 0.0079999999999999099609 rpy=3.925487559252586102e-15 1.0310330126129698141e-14 2.1281244330296900102, axis 0 0 1, limit effort=1 velocity=20
- added joint wheel_d: type revolute, parent lim_frame, child wheel_shaft_2, origin xyz=-0.11099999999999919653 8.8817841970012523234e-16 0.0079999999999987997379 rpy=-6.7482963394882867293e-15 9.8290467948461433558e-15 0.99854103579698927362, axis 0 0 1, limit effort=1 velocity=20
